Commit message: Working optimization

File: example/atlas/urdf/atlas_simple_contact_noback.urdf (robot description, URDF)
Before this commit: robot atlas, 16 links, 15 joints
Joints:
- joint l_leg_akx: limit lower=-0.8 upper=0.8 effort=130 velocity=12 -> lower=-0.8 upper=0.8 effort=150 velocity=12
- joint l_leg_aky: limit lower=-1.3 upper=1 effort=70 velocity=12 -> lower=-1.3 upper=1 effort=190 velocity=12
- joint r_leg_akx: limit lower=-0.8 upper=0.8 effort=130 velocity=12 -> lower=-0.8 upper=0.8 effort=150 velocity=12
- joint r_leg_aky: limit lower=-1.3 upper=1 effort=70 velocity=12 -> lower=-1.3 upper=1 effort=190 velocity=12

Commit message: Updated the ATLAS example.

File: example/atlas/urdf/atlas_simple_contact_noback.urdf (robot description, URDF)
Before this commit: robot atlas, 16 links, 15 joints
Joints:
- joint l_leg_kny: limit lower=0 upper=2.38569 effort=220 velocity=12 -> lower=0.1 upper=2.38569 effort=220 velocity=12
- joint r_leg_kny: limit lower=0 upper=2.38569 effort=220 velocity=12 -> lower=0.1 upper=2.38569 effort=220 velocity=12
